Commit message: SLAM MAP Creation plus pozitioning + nav2 working withouth hacks

File: src/carucior_asamblat/urdf/carucior_asamblat.urdf (robot description, URDF)
Before this commit: robot carucior_asamblat, 8 links, 7 joints
Links:
- added link base_footprint
- link roata_fata_dreapta: geometry collision cylinder length=0.10 radius=0.12; visual mesh filename=package://carucior_asamblat/meshes/roata_fata_dreapta.STL
- link roata_fata_stanga: geometry collision cylinder length=0.10 radius=0.12; visual mesh filename=package://carucior_asamblat/meshes/roata_fata_stanga.STL
- link roata_spate_dreapta: geometry collision cylinder length=0.10 radius=0.12; visual mesh filename=package://carucior_asamblat/meshes/roata_spate_dreapta.STL
- link roata_spate_stanga: geometry collision cylinder length=0.10 radius=0.12; visual mesh filename=package://carucior_asamblat/meshes/roata_spate_stanga.STL
Joints:
- added joint base_footprint_to_base_link: type fixed, parent base_footprint, child base_link, origin xyz=-0.24 -0.51 -0.24 rpy=0 0 1.5708
- joint left_back_wheel: axis 0 0 1 -> 0 0 -1
- joint left_front_wheel: axis 0 0 1 -> 0 0 -1
- joint right_back_wheel: axis 0 0 -1 -> 0 0 1
- joint right_front_wheel: axis 0 0 -1 -> 0 0 1

Commit message: merge urmarirea omului

File: src/carucior_asamblat/urdf/carucior_asamblat.urdf (robot description, URDF)
Before this commit: robot carucior_asamblat, 9 links, 8 joints
Links:
- added link lidar_legs, mass 0.05; collision cylinder length=0.04 radius=0.03
Joints:
- added joint lidar_legs_joint: type fixed, parent base_footprint, child lidar_legs, origin xyz=0.55 0.0 0.30 rpy=0 0 0
